Commit message: fix urdf file

File: robot_description/description/lidar.xacro (robot description, xacro)
@@ -4,5 +4,5 @@
         <parent link="chassis"/>
         <child link="lidar_link"/>
-        <origin xyz="0.45 0.0 0.16" rpy="0 0 0"/>
+        <origin xyz="0.35 0.0 0.245" rpy="0 0 0"/>
     </joint>
     <link name="lidar_link">

File: robot_description/description/robot_core.xacro (robot description, xacro)
@@ -30,18 +30,18 @@
         <parent link="base_link" />
         <child link="chassis" />
-        <origin xyz="-0.25 0.0 0.0" rpy="0.0 0.0 0.0" />
+        <origin xyz="-0.2 0.0 0.0" rpy="0.0 0.0 0.0" />
     </joint>
     <link name="chassis">
         <visual>
-            <origin xyz="0.25 0 0.075"/>
+            <origin xyz="0.2 0 0.1"/>
             <geometry>
-                <box size="0.5 0.3 0.12"/>
+                <box size="0.4 0.3 0.245"/>
             </geometry>
             <material name="white"/>
         </visual>
         <collision>
-            <origin xyz="0.25 0 0.075"/>
+            <origin xyz="0.2 0 0.1"/>
             <geometry>
-                <box size="0.5 0.3 0.12"/>
+                <box size="0.4 0.3 0.245"/>
             </geometry>
         </collision>
@@ -54,5 +54,5 @@
         <parent link="base_link" />
         <child link="left_wheel_2" />
-        <origin xyz="-0.125 0.175 0" rpy="-${pi/2} 0 0" />
+        <origin xyz="-0.13 0.175 0" rpy="-${pi/2} 0 0" />
         <axis xyz="0 0 1"/>
     </joint>
@@ -77,5 +77,5 @@
         <parent link="base_link" />
         <child link="left_wheel_1" />
-        <origin xyz="0.125 0.175 0" rpy="-${pi/2} 0 0" />
+        <origin xyz="0.13 0.175 0" rpy="-${pi/2} 0 0" />
         <axis xyz="0 0 1"/>
     </joint>
@@ -100,5 +100,5 @@
         <parent link="base_link" />
         <child link="right_wheel_2" />
-        <origin xyz="-0.125 -0.175 0" rpy="${-pi/2} 0 0" />
+        <origin xyz="-0.13 -0.175 0" rpy="${-pi/2} 0 0" />
         <axis xyz="0 0 1"/>
     </joint>
@@ -123,5 +123,5 @@
         <parent link="base_link" />
         <child link="right_wheel_1" />
-        <origin xyz="0.125 -0.175 0" rpy="${-pi/2} 0 0" />
+        <origin xyz="0.13 -0.175 0" rpy="${-pi/2} 0 0" />
         <axis xyz="0 0 1"/>
     </joint>
